File: schematic.sch (EAGLE design)
At the start: 0 parts

Commit message: .
Parts:
- added C1: (no value), rcl:C-EUC0402
- added F1: 0.5A, rcl:R-EU_R0402
- added P1: TYPE-C-16PIN, usb:TYPE-C-16PIN
- added Q1: (no value), library:CJ2301
- added U1: ME6211C33M5G, library:ME6211C33M5G
Connections:
- new net D_N: P1.A7, P1.B7
- new net D_P: P1.A6, P1.B6
- new net GND: P1.A1, P1.A12, P1.B1, P1.B12
- new net N$2: Q1.2, U1.VIN
- new net VBAT: Q1.3
- new net VBUS: F1.2, P1.A4, P1.A9, P1.B4, P1.B9

Commit message: .
Parts:
- added C113, C5, C7: 100nF, rcl:C-EUC0402
- added C13, C3, C4: 1uF, rcl:C-EUC0402
- added C2: 10uF, rcl:C-EUC0402
- added D2: CESD5V0D1, Diodes:CESD5V0D1
- added IC1: CP2102, silabs:CP2102
- added R3, R4: 100k, rcl:R-EU_R0402
- added SJ2: (no value), jumper:SJ
- added U4: ESP8266, Espressif:ESP8266
- C1: value (none) -> 1uF
Connections:
- removed net N$2: Q1.2, U1.VIN
- new net +3V3: C13.1, C2.1, C7.1, U4.VDD, U4.VDD3P3@1, U4.VDD3P3@2, U4.VDDA@1, U4.VDDA@2, U4.VDDPST@1, U4.VDDPST@2
- new net +5V: D2.A, F1.1, Q1.1, R3.2
- new net DTR: IC1.DTR
- new net EN: R4.2, SJ2.2, U1.CE
- new net N$1: C113.1, IC1.VDD
- new net POWER: C4.2, C5.2, IC1.REGIN, IC1.VBUS
- new net RTS: IC1.RTS
- new net RX: IC1.TXD
- new net TX: IC1.RXD
- new net VIN: C1.1, C3.1, D2.C, Q1.2, R4.1, U1.VIN, U1.VOUT
- net D_N: now also IC1.D-
- net D_P: now also IC1.D+
- net GND: now also C1.2, C113.2, C13.2, C2.2, C3.2, C4.1, C5.1, C7.2, IC1.GND, IC1.GND@EXP, IC1.GND@M, R3.1, SJ2.1, U1.VSS
Other:
- moved on the sheet: C1, Q1, U1

Commit message: .
Parts:
- added ANT1: AN9520-245, antenna:AN9520-245
- added C10: 5.6pF, rcl:C-EUC0402
- added C11, C12: 10pF, rcl:C-EUC0402
- added C9: 100nF, rcl:C-EUC0402
- added K1: RESET, alps:SKSCLDE010
- added LED1: CHIP-FLAT-G_0402, LED:CHIP-FLAT-G_0402
- added R10, R11, R13, R5, R6, R7: 12k, rcl:R-EU_R0402
- added R14: 200, rcl:R-EU_R0402
- added R16: 0, rcl:R-EU_R0603
- added R18: 470, rcl:R-EU_R0402
- added R9: 2k, rcl:R-EU_R0402
- added Y2: 26MHz, crystal:YSX321SL
Connections:
- removed net POWER: C4.2, C5.2, IC1.REGIN, IC1.VBUS
- new net ADC: U4.TOUT
- new net GPIO0: R10.1, U4.GPIO0
- new net GPIO12: U4.MTDI
- new net GPIO13: U4.MTCK
- new net GPIO14: U4.MTMS
- new net GPIO15: U4.MTDO
- new net GPIO16: U4.XPD_DCDC
- new net GPIO2: LED1.C, R11.1, U4.GPIO2
- new net GPIO4/SDA: U4.GPIO4
- new net GPIO5/SCL: U4.GPIO5
- new net LNA: C10.1, U4.LNA
- new net N$10: ANT1.FEED_TERMINATION, R16.2
- new net N$11: LED1.A, R9.1
- new net N$2: C12.2, U4.XTALI, Y2.P$2
- new net N$3: C11.2, U4.XTALO, Y2.P$1
- new net N$4: R13.2, U4.RES12K
- new net N$5: R7.2, U4.EN
- new net N$7: C10.2, R16.1
- new net N$8: R14.1, U4.SD_CLK
- new net N$9: R18.1, U4.UTXD0
- new net RST: C9.1, K1.1, K1.2, R5.1, R6.2, U4.EXT_RSTB
- new net SD_CLK: R14.2
- new net SD_CS0: U4.SD_CMD
- new net SD_HD: U4.SD_D2
- new net SD_SI: U4.SD_D1
- new net SD_SO: U4.SD_D0
- new net SD_WP: U4.SD_D3
- net +3V3: now also C1.1, R10.2, R11.2, R6.1, R7.1, R9.2, U1.VOUT
- net +5V: now also C4.2, C5.2, IC1.REGIN, IC1.VBUS
- net GND: now also C11.1, C12.1, C9.2, K1.3, K1.4, R13.1, R5.2, U4.GND
- net RX: now also U4.URXD0
- net TX: now also R18.2
- net VIN: no longer C1.1, U1.VOUT
