File: wemos_d1_mini_pro.sch (EAGLE design)
At the start: 28 parts, among them IC1 CP2102, P1 TYPE-C-16PIN, U1 ME6211C33M5G, U4 ESP8266, Y2 26MHz

Commit message: .
Parts:
- added C17, C9: 100nF, rcl:C-EUC0402
- added C6, C8: 10uF, rcl:C-EUC0402
- added K1: RESET, alps:SKSCLDE010
- added LED1: CHIP-FLAT-G_0402, LED:CHIP-FLAT-G_0402
- added LED2: CHIP-FLAT-R_0402, LED:CHIP-FLAT-R_0402
- added R1: 220k, rcl:R-EU_R0402
- added R10, R11, R5: 12k, rcl:R-EU_R0402
- added R12, R8, R9: 2k, rcl:R-EU_R0402
- added R16: 0, rcl:R-EU_R0603
- added R17: 130k, rcl:R-EU_R0402
- added R19: 470, rcl:R-EU_R0402
- added R2: 100k, rcl:R-EU_R0402
- added SJ1, SJ3: (no value), jumper:SJ
- added U2: UMH3N, UMH3N:UMH3N
- added U5: W25Q128JVPIQ, flash:W25Q128JVPIQ
- added U6: TP4054-42-SOT25-R, TP4054-42-SOT25-R:TP4054-42-SOT25-R
- Y2: value 26MHz -> (none); SPICEPREFIX B -> (none)
Connections:
- new net A0: R1.2, SJ1.2
- new net N$10: ANT1.FEED_TERMINATION, R16.2
- new net N$11: LED1.A, R9.1
- new net N$12: LED2.A, R8.1
- new net N$13: LED2.C, U6.!CHRG
- new net N$14: R17.2, SJ1.1
- new net N$16: R19.2, SJ3.1
- new net RST: C9.1, K1.1, K1.2, R19.1, R5.1, R6.2, U2.C1, U4.EXT_RSTB
- net +3V3: now also C17.1, R10.2, R11.2, R9.2, U5.VCC
- net ADC: now also R1.1, R2.2
- net DTR: now also U2.B1, U2.E2
- net GND: now also C17.2, C6.2, C8.2, C9.2, K1.3, K1.4, R12.1, R2.1, R5.2, U5.GND_1, U5.GND_2, U6.GND
- net GPIO0: now also R10.1, U2.C2
- net GPIO16: now also SJ3.2
- net GPIO2: now also LED1.C, R11.1
- net N$2: now also Y2.P$1; no longer Y2.P$2
- net N$3: now also Y2.P$2; no longer Y2.P$1
- net N$6: now also R12.2, U6.PROG; no longer R6.2, U4.EXT_RSTB
- net N$7: now also R16.1; no longer ANT1.FEED_TERMINATION
- net RTS: now also U2.B2, U2.E1
- net SD_CLK: now also U5.CLK
- net SD_CS0: now also U5.!CS
- net SD_HD: now also U5.IO3
- net SD_SI: now also U5.DI(IO0)
- net SD_SO: now also U5.DO(IO1)
- net SD_WP: now also U5.IO2
- net VBAT: now also C6.1, R17.1, U6.BAT
- net VBUS: now also C8.1, R8.2, U6.VCC
Other:
- moved on the sheet: ANT1, C1, C10, C11, C113, C12, C13, C2, C3, C4, C5, C7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
