File: wemos_d1_mini_pro.sch (EAGLE design)
At the start: 51 parts, among them IC1 CP2102, K1 RESET, P1 TYPE-C-16PIN, U1 ME6211C33M5G, U2 UMH3N, U4 ESP8266, U5 W25Q128JVPIQ, U6 TP4054-42-SOT25-R

Commit message: .
Parts:
- added J1, J2: M08X1, Connectors:M08X1
- added U$1: ZH1.25, Connectors:ZH1.25
- R16: device rcl:R-EU_R0603 -> rcl:R-EU_R0402
Connections:
- net +3V3: now also J1.8
- net +5V: now also J2.8
- net A0: now also J1.2
- net GND: now also J2.7, U$1.2
- net GPIO0: now also J2.5
- net GPIO12: now also J1.5
- net GPIO13: now also J1.6
- net GPIO14: now also J1.4
- net GPIO15: now also J1.7
- net GPIO16: now also J1.3
- net GPIO2: now also J2.6
- net GPIO4/SDA: now also J2.4
- net GPIO5/SCL: now also J2.3
- net RST: now also J1.1
- net RX: now also J2.2
- net TX: now also J2.1
- net VBAT: now also U$1.1
Changed lines of the file:
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@@
 <part name="R14" library="rcl" library_urn="urn:adsk.eagle:library:334" deviceset="R-EU_" device="R0402" package3d_urn="urn:adsk.eagle:package:23547/3" value="200"/>
 <part name="R18" library="rcl" library_urn="urn:adsk.eagle:library:334" deviceset="R-EU_" device="R0402" package3d_urn="urn:adsk.eagle:package:23547/3" value="470"/>
-<part name="R16" library="rcl" library_urn="urn:adsk.eagle:library:334" deviceset="R-EU_" device="R0603" package3d_urn="urn:adsk.eagle:package:23555/3" value="0"/>
+<part name="R16" library="rcl" library_urn="urn:adsk.eagle:library:334" deviceset="R-EU_" device="R0402" package3d_urn="urn:adsk.eagle:package:23547/3" value="0"/>
 <part name="R10" library="rcl" library_urn="urn:adsk.eagle:library:334" deviceset="R-EU_" device="R0402" package3d_urn="urn:adsk.eagle:package:23547/3" value="12k"/>
 <part name="R11" library="rcl" library_urn="urn:adsk.eagle:library:334" deviceset="R-EU_" device="R0402" package3d_urn="urn:adsk.eagle:package:23547/3" value="12k"/>
@@
 <part name="SJ3" library="jumper" library_urn="urn:adsk.eagle:library:252" deviceset="SJ" device="" package3d_urn="urn:adsk.eagle:package:15471/1"/>
 <part name="FRAME1" library="frames" library_urn="urn:adsk.eagle:library:229" deviceset="DINA3_L" device=""/>
+<part name="U$1" library="Connectors" library_urn="urn:adsk.eagle:library:25488128" deviceset="ZH1.25" device="" package3d_urn="urn:adsk.eagle:package:25488131/1"/>
+<part name="J1" library="Connectors" deviceset="M08X1" device=""/>
+<part name="J2" library="Connectors" deviceset="M08X1" device=""/>
 </parts>
 <sheets>
@@
 <attribute name="SHEET" x="373.38" y="1.27" size="2.54" layer="94"/>
 <attribute name="DRAWING_NAME" x="304.8" y="19.05" size="2.54" layer="94"/>
+</instance>
+<instance part="U$1" gate="G$1" x="109.22" y="76.2" smashed="yes"/>
+<instance part="J1" gate="G$1" x="289.56" y="87.63" smashed="yes">
+<attribute name="NAME" x="287.655" y="98.425" size="1.27" layer="95"/>
+<attribute name="VALUE" x="287.655" y="75.565" size="1.27" layer="96"/>
+</instance>
+<instance part="J2" gate="G$1" x="335.28" y="87.63" smashed="yes">
+<attribute name="NAME" x="333.375" y="98.425" size="1.27" layer="95"/>
+<attribute name="VALUE" x="333.375" y="75.565" size="1.27" layer="96"/>
 </instance>
 </instances>
@@
 <pinref part="GND23" gate="1" pin="GND"/>
 <wire x1="22.86" y1="40.64" x2="22.86" y2="35.56" width="0.1524" layer="91"/>
+</segment>
+<segment>
+<pinref part="U$1" gate="G$1" pin="2"/>
+<wire x1="101.6" y1="78.74" x2="99.06" y2="78.74" width="0.1524" layer="91"/>
+<label x="93.98" y="78.74" size="1.778" layer="95"/>
+</segment>
+<segment>
+<wire x1="330.2" y1="81.28" x2="327.66" y2="81.28" width="0.1524" layer="91"/>
+<pinref part="J2" gate="G$1" pin="7"/>
+<label x="327.66" y="81.28" size="1.778" layer="95" align="bottom-right"/>
 </segment>
 </net>
@@
 <pinref part="P+2" gate="1" pin="+5V"/>
 </segment>
+<segment>
+<wire x1="330.2" y1="78.74" x2="327.66" y2="78.74" width="0.1524" layer="91"/>
+<pinref part="J2" gate="G$1" pin="8"/>
+<label x="327.66" y="78.74" size="1.778" layer="95" align="bottom-right"/>
+</segment>
 </net>
 <net name="N$1" class="0">
@@
 <label x="291.846" y="204.47" size="1.778" layer="95"/>
 </segment>
+<segment>
+<wire x1="330.2" y1="93.98" x2="327.66" y2="93.98" width="0.1524" layer="91"/>
+<pinref part="J2" gate="G$1" pin="2"/>
+<label x="327.66" y="93.98" size="1.778" layer="95" align="bottom-right"/>
+</segment>
 </net>
 <net name="TX" class="0">
@@
 <wire x1="315.722" y1="201.93" x2="316.992" y2="201.93" width="0.1524" layer="91"/>
 <label x="317.246" y="201.93" size="1.778" layer="95"/>
+</segment>
+<segment>
+<wire x1="327.66" y1="96.52" x2="330.2" y2="96.52" width="0.1524" layer="91"/>
+<pinref part="J2" gate="G$1" pin="1"/>
+<label x="327.66" y="96.52" size="1.778" layer="95" align="bottom-right"/>
 </segment>
 </net>
@@
 <wire x1="231.14" y1="111.76" x2="231.14" y2="116.84" width="0.1524" layer="91"/>
 </segment>
+<segment>
+<pinref part="J1" gate="G$1" pin="8"/>
+<wire x1="284.48" y1="78.74" x2="281.94" y2="78.74" width="0.1524" layer="91"/>
+<label x="281.94" y="78.74" size="1.778" layer="95" align="bottom-right"/>
+</segment>
 </net>
 <net name="VBAT" class="0">
@@
 <wire x1="30.48" y1="71.12" x2="30.48" y2="50.8" width="0.1524" layer="91"/>
 <junction x="30.48" y="50.8"/>
+</segment>
+<segment>
+<pinref part="U$1" gate="G$1" pin="1"/>
+<wire x1="101.6" y1="73.66" x2="99.06" y2="73.66" width="0.1524" layer="91"/>
+<label x="93.98" y="73.66" size="1.778" layer="95"/>
 </segment>
 </net>
@@
 <label x="205.74" y="38.1" size="1.778" layer="95"/>
 </segment>
+<segment>
+<pinref part="J1" gate="G$1" pin="1"/>
+<wire x1="284.48" y1="96.52" x2="281.94" y2="96.52" width="0.1524" layer="91"/>
+<label x="281.94" y="96.52" size="1.778" layer="95" align="bottom-right"/>
+</segment>
 </net>
 <net name="LNA" class="0">
@@
 <label x="241.3" y="38.1" size="1.778" layer="95"/>
 </segment>
+<segment>
+<pinref part="J1" gate="G$1" pin="3"/>
+<wire x1="284.48" y1="91.44" x2="281.94" y2="91.44" width="0.1524" layer="91"/>
+<label x="281.94" y="91.44" size="1.778" layer="95" align="bottom-right"/>
+</segment>
 </net>
 <net name="SD_SO" class="0">
@@
 <label x="292.1" y="222.25" size="1.778" layer="95"/>
 </segment>
+<segment>
+<pinref part="J1" gate="G$1" pin="4"/>
+<wire x1="284.48" y1="88.9" x2="281.94" y2="88.9" width="0.1524" layer="91"/>
+<label x="281.94" y="88.9" size="1.778" layer="95" align="bottom-right"/>
+</segment>
 </net>
 <net name="GPIO12" class="0">
@@
 <label x="292.1" y="219.71" size="1.778" layer="95"/>
 </segment>
+<segment>
+<pinref part="J1" gate="G$1" pin="5"/>
+<wire x1="284.48" y1="86.36" x2="281.94" y2="86.36" width="0.1524" layer="91"/>
+<label x="281.94" y="86.36" size="1.778" layer="95" align="bottom-right"/>
+</segment>
 </net>
 <net name="GPIO13" class="0">
@@
 <label x="292.1" y="217.17" size="1.778" layer="95"/>
 </segment>
+<segment>
+<pinref part="J1" gate="G$1" pin="6"/>
+<wire x1="284.48" y1="83.82" x2="281.94" y2="83.82" width="0.1524" layer="91"/>
+<label x="281.94" y="83.82" size="1.778" layer="95" align="bottom-right"/>
+</segment>
 </net>
 <net name="GPIO15" class="0">
@@
 <wire x1="289.56" y1="214.63" x2="291.846" y2="214.63" width="0.1524" layer="91"/>
 <label x="292.1" y="214.63" size="1.778" layer="95"/>
+</segment>
+<segment>
+<pinref part="J1" gate="G$1" pin="7"/>
+<wire x1="284.48" y1="81.28" x2="281.94" y2="81.28" width="0.1524" layer="91"/>
+<label x="281.94" y="81.28" size="1.778" layer="95" align="bottom-right"/>
 </segment>
 </net>
@@
 <label x="129.54" y="35.56" size="1.778" layer="95"/>
 </segment>
+<segment>
+<wire x1="330.2" y1="86.36" x2="327.66" y2="86.36" width="0.1524" layer="91"/>
+<pinref part="J2" gate="G$1" pin="5"/>
+<label x="327.66" y="86.36" size="1.778" layer="95" align="bottom-right"/>
+</segment>
 </net>
 <net name="GPIO2" class="0">
@@
 <label x="312.42" y="124.714" size="1.778" layer="95"/>
 </segment>
+<segment>
+<wire x1="330.2" y1="83.82" x2="327.66" y2="83.82" width="0.1524" layer="91"/>
+<pinref part="J2" gate="G$1" pin="6"/>
+<label x="327.66" y="83.82" size="1.778" layer="95" align="bottom-right"/>
+</segment>
 </net>
 <net name="GPIO4/SDA" class="0">
@@
 <label x="291.846" y="193.04" size="1.778" layer="95"/>
 </segment>
+<segment>
+<wire x1="330.2" y1="88.9" x2="327.66" y2="88.9" width="0.1524" layer="91"/>
+<pinref part="J2" gate="G$1" pin="4"/>
+<label x="327.66" y="88.9" size="1.778" layer="95" align="bottom-right"/>
+</segment>
 </net>
 <net name="GPIO5/SCL" class="0">
@@
 <wire x1="289.56" y1="190.5" x2="291.592" y2="190.5" width="0.1524" layer="91"/>
 <label x="291.846" y="190.5" size="1.778" layer="95"/>
+</segment>
+<segment>
+<wire x1="330.2" y1="91.44" x2="327.66" y2="91.44" width="0.1524" layer="91"/>
+<pinref part="J2" gate="G$1" pin="3"/>
+<label x="327.66" y="91.44" size="1.778" layer="95" align="bottom-right"/>
 </segment>
 </net>
@@
 <junction x="63.5" y="50.8"/>
 <label x="71.12" y="50.8" size="1.778" layer="95"/>
+</segment>
+<segment>
+<pinref part="J1" gate="G$1" pin="2"/>
+<wire x1="284.48" y1="93.98" x2="281.94" y2="93.98" width="0.1524" layer="91"/>
+<label x="281.94" y="93.98" size="1.778" layer="95" align="bottom-right"/>
 </segment>
 </net>
@@
 for full support of SPICE simulation.
 </note>
+<note version="9.0" severity="warning">
+Since Version 9.0, EAGLE supports the align property for labels.
+Labels in schematic will not be understood with this version. Update EAGLE to the latest version
+for full support of labels.
+</note>
 </compatibility>
